File: pcbs/5_switch_column/5_switch_column.sch (KiCad schematic (older format))
At the start: 6 parts, among them U1 6PinHeader

Commit message: Clean up these stinking projec files _again_
Parts:
- S1, S2, S3, S4, S5: symbol 5_switch_column-rescue:CherryMXDiode-project -> symbols:CherryMXDiode
- U1: symbol 5_switch_column-rescue:6PinHeader-project -> symbols:6PinHeader
Changed lines of the file:
@@
 	4300 5900 4500 5900
 $Comp
-L 5_switch_column-rescue:CherryMXDiode-project S1
+L symbols:CherryMXDiode S1
 U 1 1 5F2D8ACD
 P 4700 3450
@@
 $EndComp
 $Comp
-L 5_switch_column-rescue:CherryMXDiode-project S2
+L symbols:CherryMXDiode S2
 U 1 1 5F27C6D7
 P 4700 4050
@@
 $EndComp
 $Comp
-L 5_switch_column-rescue:CherryMXDiode-project S3
+L symbols:CherryMXDiode S3
 U 1 1 5F27CC87
 P 4700 4650
@@
 $EndComp
 $Comp
-L 5_switch_column-rescue:CherryMXDiode-project S4
+L symbols:CherryMXDiode S4
 U 1 1 5F27D1C8
 P 4700 5250
@@
 $EndComp
 $Comp
-L 5_switch_column-rescue:CherryMXDiode-project S5
+L symbols:CherryMXDiode S5
 U 1 1 5F27D70F
 P 4700 5850
@@
 	4900 5200 4900 5300
 $Comp
-L 5_switch_column-rescue:6PinHeader-project U1
+L symbols:6PinHeader U1
 U 1 1 5F27F443
 P 4000 3000
